File: JIStastic/JIStastic.sch (KiCad schematic (older format))
At the start: 160 parts, among them J1 ISP Header, SW1 ESC, SW10 A, SW11 Z, SW12 1.25UOPT, SW13 OPT, SW14 2, SW15 W, SW16 S, SW17 X, SW18 WIN, SW19 3, SW2 TAB, SW20 E, SW21 D, SW22 C, SW23 4, SW24 R, SW25 F, SW26 V, SW27 7USPACE, SW28 .., SW29 5, SW3 CONTROL, SW30 T, SW31 G, SW32 B, SW33 4.5USPACE, SW34 6, SW35 Y, SW36 H, SW37 N, SW38 1UKANA, SW39 1.25UKANA, SW4 SHIFT, SW41 7, SW42 U, SW43 J, SW44 M, SW45 1.5UWIN, SW46 1.25UWIN, SW47 8, SW48 I, SW49 K, SW5 FN, SW50 <, SW51 LEFT, SW52 9, SW53 O, SW54 L, SW55 >, SW56 RIGHT, SW57 0, SW58 P, SW59 :, SW6 1.25FN, SW60 /, SW61 DOWN, SW62 -, SW63 @, SW64 ], SW65 -, SW66 UP, SW67 ^, SW68 [, SW69 ENTER, SW7 RESET, SW70 SHIFT, SW71 2.75USHIFT, SW72 YEN, SW73 /, SW74 BKSP, SW75 BKSP, SW76 CLEAR, SW77 7, SW78 4, SW79 1, SW8 1, SW80 2U0, SW81 0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

Commit message: 12/21
Parts:
- SW7: symbol kbd:SW_PUSH -> JIStastic-rescue:SW_PUSH-kbd
- U1: symbol keebio:PRTR5V0U2X -> JIStastic-rescue:PRTR5V0U2X-keebio
- USB1: symbol keebio:HRO-TYPE-C-31-M-12 -> JIStastic-rescue:HRO-TYPE-C-31-M-12-keebio
Changed lines of the file:
@@
 $EndComp
 $Comp
-L keebio:HRO-TYPE-C-31-M-12 USB1
+L JIStastic-rescue:HRO-TYPE-C-31-M-12-keebio USB1
 U 1 1 61897B4A
 P 1950 14450
@@
 $EndComp
 $Comp
-L keebio:PRTR5V0U2X U1
+L JIStastic-rescue:PRTR5V0U2X-keebio U1
 U 1 1 61898C05
 P 3900 14825
@@
 $EndComp
 $Comp
-L kbd:SW_PUSH SW7
+L JIStastic-rescue:SW_PUSH-kbd SW7
 U 1 1 61899E47
 P 2775 9625
